File: Papilio_Benchy.sch (EAGLE design)
At the start: 90 parts, among them SW1 EVQQ2, U1 93C46B, U2 LTC3419EMS, U3 FT2232D, U5 ARDUINO_MEGA_SHIELD, X1 6MHz

Commit message: FT2232H upgrade
Parts:
- removed C11, C3, C4, C5, C7, C9: 0.1uF, Bogdan_Commons:C0805
- removed C12, C6: 27pF, Bogdan_Commons:C0805
- removed R1: 10K, Bogdan_Commons:R0805
- removed R10, R11, R8: 68, GadgetFactory:R0805
- removed R12, R13: 220, GadgetFactory:R0805
- removed R2, R6: 27R, Bogdan_Commons:R0805
- removed R3: 1K5, Bogdan_Commons:R0805
- removed R4: 2K2, Bogdan_Commons:R0805
- removed R7: 470R, Bogdan_Commons:R0805
- removed RX, TX: (no value), led:LEDCHIP-LED0805
- removed U1: 93C46B, Bogdan_Commons:DIGITAL-EEPROM-MICROWIRE-6P_SOT23
- removed U3: FT2232D, Bogdan_Commons:FT2232D
- removed USB: MINI-USB-32005-201, con-cypressindustries:MINI-USB-32005-201
- removed X1: 6MHz, crystal:CRYSTALHC49S
- added C1: 3.3uF, dp_devices:CAP_POLSMC_A
- added C10, C8: 27pF, dp_devices:CAPC805
- added C14, C32: 4.7uF, dp_devices:CAP_POLSMC_A
- added C2, C33, C34, C35, C36, C37, C38, C39, C40, C41: 0.1uF, dp_devices:CAPC805
- added CONN1: CONN_USB, dp_devices:CONN_USB
- added IC1: FT2232H, DP-EagleLibrary:FT2232H
- added IC2: 93C46, dp_devices:93C46
- added L4, L5: (no value), dp_devices:FERRITE_BEAD805
- added R34, R36, R38, R39: 10k, dp_devices:RESISTORR805R805
- added R35: 2.2k, dp_devices:RESISTORR805R805
- added R40, R41: 470, dp_devices:RESISTORR805R805
- added R9: 12k 1%, dp_devices:RESISTORR805R805
- added RX1, TX1: (no value), dp_devices:LED805
- added X2: 12MHz, dp_devices:CRYSTAL_212M_
Connections:
- removed net 3V3OUT_A: C5.2, U3.3V3OUT
- removed net D+: R2A.1, USB.3
- removed net D-: R6A.1, USB.2
- removed net DO_A: R1A.2, R4A.1, U1.DO
- removed net EECS_A: U1.CS, U3.EECS
- removed net EEDATA_A: R4A.2, U1.DI, U3.EEDATA
- removed net EESK: U1.CLK, U3.EESK
- removed net FILTERED_VCC_A: C7.2, R7A.1, U3.AVCC
- removed net N$15_A: R3A.2, U3.RSTOUT#
- removed net N$2: R12A.2, RX.C
- removed net N$3: R13A.2, TX.C
- removed net N$4: R13A.1, U3.BCBUS3
- removed net N$5: R12A.1, U3.BCBUS2
- removed net USBDM_A: R6A.2, U3.USBDM
- removed net USBDP_A: R2A.2, R3A.1, U3.USBDP
- removed net USB_TCK: R11A.1, U3.ADBUS0
- removed net USB_TDI: R10A.1, U3.ADBUS1
- removed net USB_TMS: R8A.1, U3.ADBUS3
- removed net XTIN_A: C12.2, U3.XTIN, X1.2
- removed net XTOUT_A: C6.2, U3.XTOUT, X1.1
- new net !PWEREN: IC1.PWREN#
- new net !RESET: IC1.RESET#, R34.2
- new net !SUSPEND: IC1.SUSPEND#
- new net 1.8V: C1.+, C35.1, C36.1, C37.1, IC1.VCORE0, IC1.VCORE1, IC1.VCORE2, IC1.VREGOUT
- new net 3.3V: C2.1, C38.1, C39.1, C40.1, C41.1, IC1.VCCIO0, IC1.VCCIO1, IC1.VCCIO2, IC1.VCCIO3, IC1.VREGIN, IC2.ORG, IC2.VCC, L4.2, L5.2, R34.1, R36.2, R38.2, R39.2, RX1.A, TX1.A
- new net AC0: IC1.ACBUS0/TXDEN/GPIOH0
- new net AC1: IC1.ACBUS1/GPIOH1
- new net AC2: IC1.ACBUS2/GPIOH2
- new net AC3: IC1.ACBUS3/RXLED#/GPIOH3, R40.1
- new net AC4: IC1.ACBUS4/TXLED#/GPIOH4, R41.1
- new net AC5: IC1.ACBUS5/GPIOH5
- new net AC6: IC1.ACBUS6/GPIOH6
- new net AC7: IC1.ACBUS7/GPIOH7
- new net AD0: IC1.ADBUS0/TXD/TCK/SK
- new net AD1: IC1.ADBUS1/RXD/TDI/DO
- new net AD2: IC1.ADBUS2/RTS#/TDO/DI
- new net AD3: IC1.ADBUS3/CTS#/TMS/CS
- new net AD4: IC1.ADBUS4/DTR#/GPIOL0
- new net AD5: IC1.ADBUS5/DSR#/GPIOL1
- new net AD6: IC1.ADBUS6/DCD#/GPIOL2
- new net AD7: IC1.ADBUS7/RI#/GPIOL3
- new net BC0: IC1.BCBUS0/GPIOH1
- new net BC1: IC1.BCBUS1/GPIOH2
- new net BC2: IC1.BCBUS2
- new net BC3: IC1.BCBUS3/RXLED#/GPIOH3
- new net BC4: IC1.BCBUS4/TXLED#/GPIOH4
- new net BC5: IC1.BCBUS5/GPIOH5
- new net BC6: IC1.BCBUS6/GPIOH6
- new net BC7: IC1.BCBUS7/GPIOH7
- new net BD0: IC1.BDBUS0/TXD/TCK/SK
- new net BD1: IC1.BDBUS1/RXD/TDI/DO
- new net BD2: IC1.BDBUS2/RTS#/TDO/DI
- new net BD3: IC1.BDBUS3/CTS#/TMS/CS
- new net BD4: IC1.BDBUS4/DTR#/GPIOL0
- new net BD5: IC1.BDBUS5/DSR#/GPIOL1
- new net BD6: IC1.BDBUS6/DCD#/GPIOL2
- new net BD7: IC1.BDBUS7/RI#/GPIOL3
- new net DM: CONN1USB.D-, IC1.DM
- new net DP: CONN1USB.D+, IC1.DP
- new net EECLK: IC1.EECLK, IC2.SK, R36.1
- new net EECS: IC1.EECS, IC2.CS, R39.1
- new net EEDATA: IC1.EEDATA, IC2.DI, R35.2
- new net N$22: C8.1, IC1.OSCI, X2.X1
- new net N$23: C10.1, IC1.OSC0, X2.X2
- new net N$24: R40.2, RX1.C
- new net N$25: R41.2, TX1.C
- new net N$45: IC2.DO, R35.1, R38.1
- new net N$48: C32.+, C34.1, IC1.VPHY, L5.1
- new net N$49: C14.+, C33.1, IC1.VPLL, L4.1
- new net N$9: IC1.REF, R9.2
- net 3V3: no longer RX.A, TX.A, U3.SI/WUA, U3.SI/WUB, U3.VCCIOA, U3.VCCIOB
- net 5V: now also CONN1USB.VUSB
- net 5V0: no longer C11.2, C3.2, C4.2, C9.2, R1A.1, R7A.2, U1.VCC, U3.RESET#, U3.VCC@3, U3.VCC@42, USB.1
- net GND: now also C1.-, C10.2, C14.-, C2.2, C32.-, C33.2, C34.2, C35.2, C36.2, C37.2, C38.2, C39.2, C40.2, C41.2, C8.2, CONN1USB.GND, IC1.AGND, IC1.GND0, IC1.GND1, IC1.GND2, IC1.GND3, IC1.GND4, IC1.GND5, IC1.GND6, IC1.GND7, IC1.TEST, IC2.GND, R9.1; no longer C11.1, C12.1, C3.1, C4.1, C5.1, C6.1, C7.1, C9.1, U1.GND, U3.GND@18, U3.GND@25, U3.GND@34, U3.GND@9, U3.GND@ANALOG, U3.TEST, USB.5
- net TCK: no longer R11A.2
- net TDI: no longer R10A.2
- net TDO: no longer U3.ADBUS2
- net TMS: no longer R8A.2
- net USB_RXD: no longer U3.BDBUS1
- net USB_TXD: no longer U3.BDBUS0
Other:
- note removed: "93LC46B"

Commit message: Arduino Leonardo
Parts:
- added C11, C9: 22p, SmartPrj:C-EUC0603
- added C3, C4, C6: 100n, SmartPrj:C-EUC0603
- added C5, C7: 1uF, SmartPrj:C-EUC0603
- added D2: CD1206-S01575, diode:DIODE-MINIMELF
- added J1: USB MICRO, SmartPrj:MYCON2_USB-MINI-B
- added L, RX, TX: Yellow, led:LEDCHIPLED_0805
- added L6: MH2029-300Y, wuerth-elektronik:WE-CBF_0805
- added ON: Green, led:LEDCHIPLED_0805
- added R1: 1M, SmartPrj:R-EU_R0603
- added R2, R3: NM, SmartPrj:R-EU_R0402
- added R4, R6: 22R, GadgetFactory_6.0:R0805
- added R7, R8: 10K, GadgetFactory_6.0:R0805
- added RN2: 1K, resistor-dil:4R-NCAY16
- added U1: ATMEGA32U4-XUMU, SmartPrj:ATMEGA32U4-XUMU
- added U3: ATMEGA32U4-XUAU, SmartPrj:ATMEGA32U4-XUAU
- added Y1: 16MHz KX-7, SmartPrj:CRYSTAL-3.2-2.5
Connections:
- new net +5V: C3.1, C4.1, D2.C, L6.1, R7A.2, RN2A.1, RN2C.1, RN2D.1, U1.UVCC, U1.VCC, U1.VCC1, U3.UVCC, U3.VCC, U3.VCC1
- new net AGND: C6.1, R2.1, U1.GND3, U3.GND3
- new net AREF: C6.2, U1.AREF, U3.AREF
- new net AVCC: C5.1, L6.2, U1.AVCC, U1.AVCC1, U3.AVCC, U3.AVCC1
- new net D+: J1.D+, R6A.1
- new net D-: J1.D-, R4A.1
- new net D0/RX: U1.(RXD1/AIN1/INT2)PD2, U3.(RXD1/AIN1/INT2)PD2
- new net D1/TX: U1.(TXD1/INT3)PD3, U3.(TXD1/INT3)PD3
- new net D2/SDA: U1.(SDA/INT1)PD1, U3.(SDA/INT1)PD1
- new net D3/SCL: U1.(OC0B/SCL/INT0)PD0, U3.(OC0B/SCL/INT0)PD0
- new net D5*: U1.(OC3A/#0C4A)PC6, U3.(OC3A/#0C4A)PC6
- new net D6*: U1.(T0/OC4D/ADC10)PD7, U3.(T0/OC4D/ADC10)PD7
- new net HWB: R8A.2, U1.(#HWB)PE2, U3.(#HWB)PE2
- new net IO10*: U1.(PCINT6/OC1B/OC4B/ADC13)PB6, U3.(PCINT6/OC1B/OC4B/ADC13)PB6
- new net IO11*: U1.(PCINT7/OC0A/OC1C/#RTS)PB7, U3.(PCINT7/OC0A/OC1C/#RTS)PB7
- new net IO12: U1.(T1/#OC4D/ADC9)PD6, U3.(T1/#OC4D/ADC9)PD6
- new net IO13*: RN2B.1, U1.(ICP3/CLK0/OC4A)PC7, U3.(ICP3/CLK0/OC4A)PC7
- new net IO8: U1.(ADC11/PCINT4)PB4, U3.(ADC11/PCINT4)PB4
- new net IO9*: U1.(PCINT5/OC1A/#OC4B/ADC12)PB5, U3.(PCINT5/OC1A/#OC4B/ADC12)PB5
- new net MISO: U1.(PD0/MISO/PCINT3)PB3, U3.(PD0/MISO/PCINT3)PB3
- new net MOSI: U1.(PDI/MOSI/PCINT2)PB2, U3.(PDI/MOSI/PCINT2)PB2
- new net N$2: L.A, RN2B.2
- new net N$3: ON.A, RN2A.2
- new net N$4: RN2C.2, TX.A
- new net N$5: RN2D.2, RX.A
- new net RD+: R6A.2, U1.D+, U3.D+
- new net RD-: R4A.2, U1.D-, U3.D-
- new net RXLED: RX.C, U1.(SS/PCINT0)PB0, U3.(SS/PCINT0)PB0
- new net SCK: U1.(SCLK/PCINT1)PB1, U3.(SCLK/PCINT1)PB1
- new net TXLED: TX.C, U1.(XCK1/#CTS)PD5, U3.(XCK1/#CTS)PD5
- new net UCAP: C7.1, U1.UCAP, U3.UCAP
- new net UGND: C7.2, R3.2, U1.UGND, U3.UGND
- new net USBID: J1.ID
- new net VUSB: U1.VBUS, U3.VBUS
- new net XTAL1: C11.1, R1.1, U1.XTAL1, U3.XTAL1, Y1.C1
- new net XTAL2: C9.2, R1.2, U1.XTAL2, U3.XTAL2, Y1.C2
- new net XUSB: J1.VBUS
- net A0: now also U1.(ADC7/TDI)PF7, U3.(ADC7/TDI)PF7
- net A1: now also U1.(ADC6/TDO)PF6, U3.(ADC6/TDO)PF6
- net A2: now also U1.(ADC5/TMS)PF5, U3.(ADC5/TMS)PF5
- net A3: now also U1.(ADC4/TCK)PF4, U3.(ADC4/TCK)PF4
- net A4: now also U1.(ADC1)PF1, U3.(ADC1)PF1
- net A5: now also U1.(ADC0)PF0, U3.(ADC0)PF0
- net D4: now also U1.(ICP1/ADC8)PD4, U3.(ICP1/ADC8)PD4
- net D7: now also U1.(INT6/AIN0)PE6, U3.(INT6/AIN0)PE6
- net GND: now also C11.2, C3.2, C4.2, C5.2, C9.1, J1.GND, J1.SH1, J1.SH2, J1.SH3, J1.SH4, J1.SH5, J1.SH6, L.C, ON.C, R2.2, R3.1, R8A.1, U1.GND, U1.GND1, U1.GND2, U1.PAD, U3.GND, U3.GND1, U3.GND2, U3.PAD, Y1.GND@1, Y1.GND@2
- net RESET: now also D2.A, R7A.1, U1.RESET, U3.RESET
Other:
- note added: "#PWM 10bit"
- note added: "#PWM 16bit"
- note added: "#PWM 8/16bit"
- note added: "#PWM 8bit"
- note added: "#PWM Hi-Speed"
- note added: "+A10"
- note added: "+A11"
- note added: "+A6"
- note added: "+A7"
- note added: "+A8"
- note added: "+A9"
- note added: "+AIN0"
- note added: "+PWM COMPL IO10"
- note added: "0"
- note added: "1"
- note added: "10#"
- note added: "11#"
- note added: "12"
- note added: "13"
- note added: "2"
- note added: "3#"
- note added: "4"
- note added: "5#"
- note added: "6#"
- note added: "7"
- note added: "8"
- note added: "9#"
- note added: "ALT1"
- note added: "ALT2"
- note added: "ALT3"
- note added: "IO"
- note added: "PWM 16bit COMPL D6"
- note added: "TO ICSP"
- note added: "USB"
- note added: "USB boot En"

Commit message: Connections added and blocks placed.
Parts:
- removed ADC: ADC088S102CIMT, spiadc:ADC088S102CIMT
- removed C13, C20: .1uF, rcl:C-EUC0603
- removed L1: FERRITEBEAD, rcl:R-EU_R0603
- removed R8: 10K, GadgetFactory_6.0:R0805
- removed U3: ATMEGA32U4-XUAU, SmartPrj:ATMEGA32U4-XUAU
- C10, C2, C33, C34, C35, C36, C37, C38, C39, C40, C41, C8: device dp_devices:CAPC805 -> dp_devices:CAPC603
- L4, L5: device dp_devices:FERRITE_BEAD805 -> dp_devices:FERRITE_BEAD603
- R34, R35, R36, R38, R39, R40, R41, R9: device dp_devices:RESISTORR805R805 -> dp_devices:RESISTORR603
- SRAM: value IS61WV25616 -> ISSI_SRAM_8BIT; device Bogdan_Commons:DIGITAL_4MB_SRAM -> GadgetFactory:ISSI_SRAM_8BIT
Connections:
- removed net AD0: IC1.ADBUS0/TXD/TCK/SK
- removed net AD1: IC1.ADBUS1/RXD/TDI/DO
- removed net AD2: IC1.ADBUS2/RTS#/TDO/DI
- removed net AD3: IC1.ADBUS3/CTS#/TMS/CS
- removed net ADC_CS: ADC.!CS, S6B3.IO_L37N_3
- removed net BD0: IC1.BDBUS0/TXD/TCK/SK
- removed net BD1: IC1.BDBUS1/RXD/TDI/DO
- removed net BD2: IC1.BDBUS2/RTS#/TDO/DI
- removed net BD3: IC1.BDBUS3/CTS#/TMS/CS
- removed net D0/RX: U1.(RXD1/AIN1/INT2)PD2, U3.(RXD1/AIN1/INT2)PD2
- removed net D1/TX: U1.(TXD1/INT3)PD3, U3.(TXD1/INT3)PD3
- removed net D10: S6B3.IO_L1N_VREF_3, SRAM.D10
- removed net D11: S6B3.IO_L2P_3, SRAM.D11
- removed net D12: S6B3.IO_L42N_GCLK24_3, SRAM.D12
- removed net D13: S6B3.IO_L42P_GCLK25_TRDY2_3, SRAM.D13
- removed net D14: S6B3.IO_L41N_GCLK26_3, SRAM.D14
- removed net D15: S6B3.IO_L41P_GCLK27_3, SRAM.D15
- removed net D2/SDA: U1.(SDA/INT1)PD1, U3.(SDA/INT1)PD1
- removed net D3/SCL: U1.(OC0B/SCL/INT0)PD0, U3.(OC0B/SCL/INT0)PD0
- removed net D5*: U1.(OC3A/#0C4A)PC6, U3.(OC3A/#0C4A)PC6
- removed net D6*: U1.(T0/OC4D/ADC10)PD7, U3.(T0/OC4D/ADC10)PD7
- removed net D8: S6B2.IO_L64N_D9_2, SRAM.D8
- removed net D9: S6B3.IO_L1P_3, SRAM.D9
- removed net HWB: R8A.2, U1.(#HWB)PE2, U3.(#HWB)PE2
- removed net IO10*: U1.(PCINT6/OC1B/OC4B/ADC13)PB6, U3.(PCINT6/OC1B/OC4B/ADC13)PB6
- removed net IO11*: U1.(PCINT7/OC0A/OC1C/#RTS)PB7, U3.(PCINT7/OC0A/OC1C/#RTS)PB7
- removed net IO12: U1.(T1/#OC4D/ADC9)PD6, U3.(T1/#OC4D/ADC9)PD6
- removed net IO13*: RN2B.1, U1.(ICP3/CLK0/OC4A)PC7, U3.(ICP3/CLK0/OC4A)PC7
- removed net IO8: U1.(ADC11/PCINT4)PB4, U3.(ADC11/PCINT4)PB4
- removed net IO9*: U1.(PCINT5/OC1A/#OC4B/ADC12)PB5, U3.(PCINT5/OC1A/#OC4B/ADC12)PB5
- removed net MISO: U1.(PD0/MISO/PCINT3)PB3, U3.(PD0/MISO/PCINT3)PB3
- removed net MOSI: U1.(PDI/MOSI/PCINT2)PB2, U3.(PDI/MOSI/PCINT2)PB2
- removed net N$10: ADC.VA, C20.1, L1.1
- removed net NC: S6B3.IO_L51P_3
- removed net RXLED: RX.C, U1.(SS/PCINT0)PB0, U3.(SS/PCINT0)PB0
- removed net SCK: U1.(SCLK/PCINT1)PB1, U3.(SCLK/PCINT1)PB1
- removed net TCK: S6BNA.TCK, U$2.JTAG_TCK
- removed net TDI: S6BNA.TDI, U$2.JTAG_TDI
- removed net TDO: S6BNA.TDO, U$2.JTAG_TDO
- removed net TMS: S6BNA.TMS, U$2.JTAG_TMS
- removed net TXLED: TX.C, U1.(XCK1/#CTS)PD5, U3.(XCK1/#CTS)PD5
- new net A18: S6B2.IO_L64N_D9_2, SRAM.A18/NC
- new net A19: S6B3.IO_L1P_3, SRAM.A19/NC
- new net A20: S6B3.IO_L2P_3, SRAM.A20/NC
- new net AD0-JTAG_TCK: IC1.ADBUS0/TXD/TCK/SK, S6B3.IO_L51P_3, S6BNA.TCK, U$2.JTAG_TCK
- new net AD1-JTAG_TDI: IC1.ADBUS1/RXD/TDI/DO, S6B3.IO_L42P_GCLK25_TRDY2_3, S6BNA.TDI, U$2.JTAG_TDI
- new net AD2-JTAG_TDO: IC1.ADBUS2/RTS#/TDO/DI, S6BNA.TDO, U$2.JTAG_TDO
- new net AD3-JTAG_TMS: IC1.ADBUS3/CTS#/TMS/CS, S6BNA.TMS, U$2.JTAG_TMS
- new net ARDUINO_RESET: D2.A, R7A.1, S6B3.IO_L1N_VREF_3, U1.RESET
- new net ATMEGA_A0: U1.(ADC7/TDI)PF7
- new net ATMEGA_A1: U1.(ADC6/TDO)PF6
- new net ATMEGA_A2: U1.(ADC5/TMS)PF5
- new net ATMEGA_A3: U1.(ADC4/TCK)PF4
- new net ATMEGA_A4: U1.(ADC1)PF1
- new net ATMEGA_A5: U1.(ADC0)PF0
- new net ATMEGA_D0/RX: U1.(RXD1/AIN1/INT2)PD2
- new net ATMEGA_D1/TX: U1.(TXD1/INT3)PD3
- new net ATMEGA_D2/SDA: U1.(SDA/INT1)PD1
- new net ATMEGA_D3/SCL: U1.(OC0B/SCL/INT0)PD0
- new net ATMEGA_D4: U1.(ICP1/ADC8)PD4
- new net ATMEGA_D5*: U1.(OC3A/#0C4A)PC6
- new net ATMEGA_D6*: U1.(T0/OC4D/ADC10)PD7
- new net ATMEGA_D7: U1.(INT6/AIN0)PE6
- new net ATMEGA_HWB: U1.(#HWB)PE2
- new net ATMEGA_IO10*: U1.(PCINT6/OC1B/OC4B/ADC13)PB6
- new net ATMEGA_IO11*: U1.(PCINT7/OC0A/OC1C/#RTS)PB7
- new net ATMEGA_IO12: U1.(T1/#OC4D/ADC9)PD6
- new net ATMEGA_IO13*: RN2B.1, U1.(ICP3/CLK0/OC4A)PC7
- new net ATMEGA_IO8: U1.(ADC11/PCINT4)PB4
- new net ATMEGA_IO9*: U1.(PCINT5/OC1A/#OC4B/ADC12)PB5
- new net ATMEGA_MISO: U1.(PD0/MISO/PCINT3)PB3
- new net ATMEGA_MOSI: U1.(PDI/MOSI/PCINT2)PB2
- new net ATMEGA_RXLED: RX.C, U1.(SS/PCINT0)PB0
- new net ATMEGA_SCK: U1.(SCLK/PCINT1)PB1
- new net ATMEGA_TXLED: TX.C, U1.(XCK1/#CTS)PD5
- new net BD0_MPSSE_TCK: IC1.BDBUS0/TXD/TCK/SK, S6B3.IO_L42N_GCLK24_3
- new net BD1_MPSSE_TDI: IC1.BDBUS1/RXD/TDI/DO, S6B3.IO_L41P_GCLK27_3
- new net BD2_MPSSE_TDO: IC1.BDBUS2/RTS#/TDO/DI, S6B3.IO_L41N_GCLK26_3
- new net BD3_MPSSE_TMS: IC1.BDBUS3/CTS#/TMS/CS, S6B3.IO_L37N_3
- net +5V: no longer U3.UVCC, U3.VCC, U3.VCC1
- net 3V3: no longer ADC.VD, C13.1, SRAM.VDD@1, SRAM.VDD@2
- net 5V0: no longer L1.2
- net A0: no longer U1.(ADC7/TDI)PF7, U3.(ADC7/TDI)PF7
- net A1: no longer U1.(ADC6/TDO)PF6, U3.(ADC6/TDO)PF6
- net A2: no longer U1.(ADC5/TMS)PF5, U3.(ADC5/TMS)PF5
- net A3: no longer U1.(ADC4/TCK)PF4, U3.(ADC4/TCK)PF4
- net A4: no longer U1.(ADC1)PF1, U3.(ADC1)PF1
- net A5: no longer U1.(ADC0)PF0, U3.(ADC0)PF0
- net AGND: no longer U3.GND3
- net AREF: no longer U3.AREF
- net AVCC: no longer U3.AVCC, U3.AVCC1
- net D4: no longer U1.(ICP1/ADC8)PD4, U3.(ICP1/ADC8)PD4
- net D7: no longer U1.(INT6/AIN0)PE6, U3.(INT6/AIN0)PE6
- net GND: no longer ADC.AGND, ADC.DGND, C13.2, C20.2, R8A.1, SRAM.!BHE, SRAM.!BLE, U3.GND, U3.GND1, U3.GND2, U3.PAD
- net MEGA_A0: no longer ADC.AIN0
- net MEGA_A1: no longer ADC.AIN1
- net MEGA_A2: no longer ADC.AIN2
- net MEGA_A3: no longer ADC.AIN3
- net MEGA_A4: no longer ADC.AIN4
- net MEGA_A5: no longer ADC.AIN5
- net MEGA_A6: no longer ADC.AIN6
- net MEGA_A7: no longer ADC.AIN7
- net MEGA_D51: no longer ADC.DIN
- net MEGA_D52: no longer ADC.DOUT
- net MEGA_D53: no longer ADC.SCLK
- net RD+: no longer U3.D+
- net RD-: no longer U3.D-
- net RESET: no longer D2.A, R7A.1, U1.RESET, U3.RESET
- net UCAP: no longer U3.UCAP
- net UGND: no longer U3.UGND
- net VUSB: no longer U3.VBUS
- net XTAL1: no longer U3.XTAL1
- net XTAL2: no longer U3.XTAL2
Other:
- note added: "TODO: Can we use init_b?"
- note added: "TODO: Make sure to put this chips reset line under control of the FPGA with a pull up resistor."
- note added: "TODO: add LED to IO 13"
- note removed: "#PWM 10bit"
- note removed: "#PWM 16bit"
- note removed: "#PWM 8/16bit"
- note removed: "#PWM 8bit"
- note removed: "#PWM Hi-Speed"
- note removed: "+A10"
- note removed: "+A11"
- note removed: "+A6"
- note removed: "+A7"
- note removed: "+A8"
- note removed: "+A9"
- note removed: "+AIN0"
- note removed: "+PWM COMPL IO10"
- note removed: "0"
- note removed: "1"
- note removed: "10#"
- note removed: "11#"
- note removed: "12"
- note removed: "13"
- note removed: "2"
- note removed: "3#"
- note removed: "4"
- note removed: "5#"
- note removed: "6#"
- note removed: "7"
- note removed: "8"
- note removed: "9#"
- note removed: "ALT1"
- note removed: "ALT2"
- note removed: "ALT3"
- note removed: "IO"
- note removed: "PWM 16bit COMPL D6"
- note removed: "TO ICSP"
- note removed: "USB boot En"
- moved on the sheet: R40, R41, RX1, TX1

Commit message: Bunch of little changes
Parts:
- added R8: 4.7K, GadgetFactory:R0603
Connections:
- removed net ATMEGA_HWB: U1.(#HWB)PE2
- removed net ATMEGA_MISO: U1.(PD0/MISO/PCINT3)PB3
- removed net ATMEGA_MOSI: U1.(PDI/MOSI/PCINT2)PB2
- removed net ATMEGA_SCK: U1.(SCLK/PCINT1)PB1
- removed net MEGA_A0: U5.A0
- removed net MEGA_A1: U5.A1
- removed net MEGA_A2: U5.A2
- removed net MEGA_A3: U5.A3
- removed net MEGA_A4: U5.A4
- removed net MEGA_A5: U5.A5
- removed net MEGA_A6: U5.A6
- removed net MEGA_A7: U5.A7
- removed net N$11: R15A.2, U5.*D3
- removed net N$12: R16A.2, U5.D4
- removed net N$13: R17A.2, U5.D5
- removed net N$14: R18A.2, U5.D6
- removed net N$15: R19A.2, U5.D7
- removed net N$16: R20A.2, U5.D8
- removed net N$17: R21A.2, U5.D9
- removed net N$18: R22A.2, U5.D10
- removed net N$19: R23A.2, U5.D11
- removed net N$20: R24A.2, U5.D12
- removed net N$21: R25A.2, U5.D13
- removed net N$6: R14A.2, U5.*D2
- removed net USB_RXD: R26A.2, U5.TX
- removed net USB_TXD: R27A.2, U5.RX
- new net NC1: S6B3.IO_L42P_GCLK25_TRDY2_3
- new net NC2: S6B3.IO_L51P_3
- net 3V3: now also R8A.2
- net 5V0: no longer U5.5V@1, U5.5V@2
- net AD0-JTAG_TCK: no longer S6B3.IO_L51P_3
- net AD1-JTAG_TDI: no longer S6B3.IO_L42P_GCLK25_TRDY2_3
- net ATMEGA_A0: now also U5.A0
- net ATMEGA_A1: now also U5.A1
- net ATMEGA_A2: now also U5.A2
- net ATMEGA_A3: now also U5.A3
- net ATMEGA_A4: now also U5.A4
- net ATMEGA_A5: now also U5.A5
- net ATMEGA_D0/RX: now also R27A.2, U5.RX
- net ATMEGA_D1/TX: now also R26A.2, U5.TX
- net ATMEGA_D2/SDA: now also R14A.2, U5.*D2
- net ATMEGA_D3/SCL: now also R15A.2, U5.*D3
- net ATMEGA_D4: now also R16A.2, U5.D4
- net ATMEGA_D5*: now also R17A.2, U5.D5
- net ATMEGA_D6*: now also R18A.2, U5.D6
- net ATMEGA_D7: now also R19A.2, U5.D7
- net ATMEGA_IO10*: now also R22A.2, U5.D10
- net ATMEGA_IO11*: now also R23A.2, U5.D11
- net ATMEGA_IO12: now also R24A.2, U5.D12
- net ATMEGA_IO13*: now also R25A.2, U5.D13
- net ATMEGA_IO8: now also R20A.2, U5.D8
- net ATMEGA_IO9*: now also R21A.2, U5.D9
- net GND: now also U1.(#HWB)PE2
- net MEGA_D51: now also U1.(SCLK/PCINT1)PB1
- net MEGA_D52: now also U1.(PDI/MOSI/PCINT2)PB2
- net MEGA_D53: now also R8A.1, U1.(PD0/MISO/PCINT3)PB3
Other:
- note added: "TODO: 5V or 3.3V power config?"
- note added: "TODO: Benchy select switch"
- note added: "TODO: Reset Line... Protect FPGA if 5V."
- note removed: "TODO: Make sure to put this chips reset line under control of the FPGA with a pull up resistor."
- moved on the sheet: SW1

Commit message: Added switch and HDMI
Parts:
- added C20: 1uF, saanlima:C0402
- added J4: HDMI-TYPE-A-RECEPTICALFCI10029449, saanlima:HDMI-TYPE-A-RECEPTICALFCI10029449
- added R10, R45: 10K, saanlima:R0402
- added R11: 0, saanlima:R0402
- added R12, R13, R42, R43: 1K, saanlima:R0402
- added R44: 100K, saanlima:R0402
- added R46: 2.2K, saanlima:R0402
- added RN1, RN3: 51, saanlima:CTS742C083
- added SW2: EVQQ2, adafruit:EVQQ2
- added T1: MOSFET-NCHANNELSMD, saanlima:MOSFET-NCHANNELSMD
- added U11: PCA9306, saanlima:PCA9306
- SW1: value EVQQ2 -> SWITCH-2CH-6P-3010010P1; device adafruit:EVQQ2 -> OPL Eagle Library:SWITCH-2CH-6P-3010010P1
Connections:
- new net DDC_SCL: J4.SCL, R42.2, U11.SCL2
- new net DDC_SDA: J4.SDA, R43.2, U11.SDA2
- new net DETECT: J4.DETECT, R10.2, R45.1
- new net FPGA_SCL: R12.2, U11.SCL1
- new net FPGA_SDA: R13.2, U11.SDA1
- new net HDMI_DET#: R46.2, T1.D
- new net N$17: R45.2, T1.G
- new net N$6: C20.1, R44.1, U11.EN, U11.VREF2
- new net SW0: S6B1.IO_L1N_VREF_1, SW1.COM2
- new net TX_HDMI_5V: J4.+5V, R11.1, R42.1, R43.1, R44.2
- net 3V3: now also R12.1, R13.1, R46.1, RN1.5, RN1.6, RN1.7, RN1.8, RN3.5, RN3.6, RN3.7, RN3.8, SW1.CH2A, U11.VREF1
- net 5V: now also R11.2
- net GND: now also C20.2, J4.CLOCKSHIELD, J4.DATA0SHIELD, J4.DATA1SHIELD, J4.DATA2SHIELD, J4.DDC/CEC-GRND, J4.RES, R10.1, SW1.CH2B, SW2.S, SW2.S1, T1.S, U11.GND; no longer SW1.S, SW1.S1
- net MEGA_D45: now also J4.DATA2+, RN1.4
- net MEGA_D46: now also J4.DATA2-, RN1.3
- net MEGA_D47: now also J4.DATA1+, RN1.2
- net MEGA_D48: now also J4.DATA1-, RN1.1
- net MEGA_D49: now also J4.CLOCK+, RN3.2
- net MEGA_D50: now also J4.CLOCK-, RN3.1
- net MEGA_D51: now also J4.DATA0+, RN3.4
- net MEGA_D52: now also J4.DATA0-, RN3.3
- net MEGA_D53: now also J4.CEC
- net RESET: now also SW2.P, SW2.P1; no longer SW1.P, SW1.P1
Other:
- note added: "Copyright Saanlima Electronics 2012"
- note added: "Do not populate"
- note added: "Saanlima Electronics"

Commit message: Schematic Cleanup - Ready for routing...
Parts:
- added R47, R48, R49: 390, GadgetFactory:R0603
Connections:
- net FPGA_RXD renamed MEGA_D1
- net FPGA_TXD renamed MEGA_D0
- removed net AD4: IC1.ADBUS4/DTR#/GPIOL0
- removed net BD4: IC1.BDBUS4/DTR#/GPIOL0
- removed net FPGA_SCL: R12.2, U11.SCL1
- removed net FPGA_SDA: R13.2, U11.SDA1
- removed net NC1: S6B3.IO_L42P_GCLK25_TRDY2_3
- removed net NC2: S6B3.IO_L51P_3
- new net AD4-DTR: IC1.ADBUS4/DTR#/GPIOL0, S6B3.IO_L42P_GCLK25_TRDY2_3
- new net BD4-DTR: IC1.BDBUS4/DTR#/GPIOL0, S6B3.IO_L51P_3
- new net N$10: R49A.2, U1.(SCLK/PCINT1)PB1
- new net N$11: R48A.2, U1.(PDI/MOSI/PCINT2)PB2
- new net N$12: R47A.2, U1.(PD0/MISO/PCINT3)PB3
- net 3V3: now also SRAM.VDD@1, SRAM.VDD@2, U5.3V3@1, U5.3V3@2, U5.3V3@3, U5.3V3@4
- net GND: now also U5.GND@5, U5.GND@6
- net MEGA_D40: now also R47A.1
- net MEGA_D41: now also R48A.1
- net MEGA_D42: now also R49A.1
- net MEGA_D43: now also R13.2, U11.SDA1
- net MEGA_D44: now also R12.2, U11.SCL1
- net MEGA_D51: no longer U1.(SCLK/PCINT1)PB1
- net MEGA_D52: no longer U1.(PDI/MOSI/PCINT2)PB2
- net MEGA_D53: no longer U1.(PD0/MISO/PCINT3)PB3
Other:
- note added: "Decoupling Caps"
- note added: "QUESTION: Reset switch control FPGA and Arduino? Or just FPGA and Arduino reset under FPGA control..."
- note added: "TODO: If this switch is too big or not practical during routing then make it smaller surface mount part or remove it."
- note removed: "Power"
- note removed: "TODO: 5V or 3.3V power config?"
- note removed: "TODO: Benchy select switch"
- note removed: "TODO: Can we use init_b?"
- note removed: "TODO: add LED to IO 13"
- note removed: "VCCO's are selectable to 1.2V, 1.5V, 1.8V, 2.5V, 3.0V, 3.3V"
- moved on the sheet: C15, C16, C17, C18, C19, C21, C22, C23, C24, C25, C26, C27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
